File: hardware/pcb/companion_carrier.kicad_pcb (KiCad board)
At the start: 2 copper layers, 44 x 104 mm, 17 parts

Commit message: Switch carrier board to all-THT/header mounting (v2)
Geoff pointed out the XIAO already carries all the MCU/USB/flash
complexity, so this board should be "just a breakout for switches and
a mic module" -- and confirmed the ordered XIAO is the pre-soldered/
header SKU, which mounts via standoff pins rather than flush reflow.
Combined with "keep the LED but make it simple THT," this became a
full mounting revision:

- XIAO: header-mounted on the carrier's BACK via its own presoldered
  pins (no separate socket needed), instead of flush castellated-SMD
  reflow on the front
- Mic: breakout module (front side, THT header), replacing the bare
  SMD chip -- matches the original breadboard-track part
- Status LED: plain THT LED + resistor, replacing the addressable
  WS2812B -- firmware now drives GPIO3 high/low instead of bit-banging
- Passives: switched to THT for consistency

Net effect: every active component is hand-solderable with a plain
iron, no reflow/hot-air anywhere. Trade-off: enclosure grew from
~14.3mm to ~22.6mm thick, since the header-mounted module needs real
standoff clearance instead of sitting flush -- called out plainly in
PHYSICAL_DESIGN_SPEC.md and the enclosure README rather than buried in
a diff.

Regenerated the PCB, enclosure, and mockup/renders to match. Flagged
hardware/ASSEMBLY_SOURCING.md and assembly_options.html as stale
(built against the old bare-SMD design) -- tracked as issue #15.

Co-Authored-By: Claude Sonnet 5 <noreply@anthropic.com>
Claude-Session: https://claude.ai/code/session_016ESUrPmzfisJUeUMDe4Dop
Parts:
- C1, C2, C3, R1: footprint carrier:R_C_0603 -> carrier:THT_passive
- D1: footprint carrier:WS2812B_5050 -> carrier:LED_3mm_THT
- MK1: footprint carrier:Knowles_SPH0645LM4H-B -> carrier:MicBreakout_SPH0645-style; moved to F.Cu
- U1: footprint carrier:XIAO-RP2040_USB-down -> carrier:XIAO-RP2040_preSoldered_header; moved to B.Cu
- moved C1 16.8 mm to (44.0, 50.0)
- moved C2 7.50 mm to (69.0, 50.0)
- moved MK1 3.50 mm to (60.0, 40.0)
Connections:
- D1 pad 1: 3V3 -> LED_A
- D1 pad 2: (no net) -> GND
- R1 pad 2: LED_DIN -> LED_A

Commit message: v2.1: revert status LED to addressable RGB (pin budget forces it)
Geoff asked for a true RGB status LED, noting it doesn't need to be
addressable. Implementing it surfaced a real constraint: a discrete
3-channel RGB LED needs 3 independent GPIOs, and the locked pin map
(docs/SPEC.md §8) leaves only 2 spares after the 9 assigned signals --
one short, with no multiplexing trick around it (charlieplexing only
saves pins when LED count exceeds pin count, not for a single 3-channel
part). Asked Geoff to choose between three resolutions; he picked
reverting to an addressable LED, since it needs only the one GPIO the
budget actually has spare.

D1 is WS2812B/SK6812-style again -- the one deliberately reintroduced
SMD part, still hand-solderable (large gull-wing pads, not a
reflow-only part like the old bare mic chip). Firmware only needs solid
colors, not animation, per the "doesn't need to be addressable" framing
-- it just turned out addressable was the only option that fit.

Regenerated PCB/mockup/renders; updated BOM.md netlist and
PHYSICAL_DESIGN_SPEC.md §7 with the full reasoning.

Co-Authored-By: Claude Sonnet 5 <noreply@anthropic.com>
Claude-Session: https://claude.ai/code/session_016ESUrPmzfisJUeUMDe4Dop
Parts:
- D1: footprint carrier:LED_3mm_THT -> carrier:WS2812B_5050
Connections:
- D1 pad 1: LED_A -> 3V3
- D1 pad 2: GND -> (no net)
- R1 pad 2: LED_A -> LED_DIN
Changed lines of the file:
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@@
   (net 12 "I2S_LRCLK")
   (net 13 "LED_DATA")
-  (net 14 "LED_A")
+  (net 14 "LED_DIN")
   (net 15 "SPARE_D9")
   (footprint "carrier:Kailh_Choc_V1" (version 20240108) (generator generate_pcb.py) (layer "F.Cu")
@@
       (net 1 "GND"))
   )
-  (footprint "carrier:LED_3mm_THT" (version 20240108) (generator generate_pcb.py) (layer "F.Cu")
+  (footprint "carrier:WS2812B_5050" (version 20240108) (generator generate_pcb.py) (layer "F.Cu")
     (at 74.0 38.0)
-    (attr through_hole)
+    (attr smd)
     (fp_text reference "D1" (at 0 -3.0) (layer "F.SilkS")
       (effects (font (size 0.8 0.8) (thickness 0.12)))
     )
-    (fp_circle (center 0 0) (end 1.5 0) (layer "F.SilkS") (width 0.12))
-    (pad "1" thru_hole circle (at -1.0 0) (size 1.4 1.4) (drill 0.8) (layers *.Cu *.Mask)
-      (net 14 "LED_A"))
-    (pad "2" thru_hole circle (at 1.0 0) (size 1.4 1.4) (drill 0.8) (layers *.Cu *.Mask)
-      (net 1 "GND"))
+    (fp_line (start -2.5 -2.5) (end 2.5 -2.5) (layer "F.SilkS") (width 0.12))
+    (fp_line (start 2.5 -2.5) (end 2.5 2.5) (layer "F.SilkS") (width 0.12))
+    (fp_line (start 2.5 2.5) (end -2.5 2.5) (layer "F.SilkS") (width 0.12))
+    (fp_line (start -2.5 2.5) (end -2.5 -2.5) (layer "F.SilkS") (width 0.12))
+    (pad "1" smd roundrect (at -2.45 -1.6) (size 1.5 1.0) (layers "F.Cu" "F.Mask" "F.Paste") (roundrect_rratio 0.25)
+      (net 2 "3V3"))
+    (pad "2" smd roundrect (at -2.45 1.6) (size 1.5 1.0) (layers "F.Cu" "F.Mask" "F.Paste") (roundrect_rratio 0.25))
+    (pad "3" smd roundrect (at 2.45 1.6) (size 1.5 1.0) (layers "F.Cu" "F.Mask" "F.Paste") (roundrect_rratio 0.25)
+      (net 1 "GND"))
+    (pad "4" smd roundrect (at 2.45 -1.6) (size 1.5 1.0) (layers "F.Cu" "F.Mask" "F.Paste") (roundrect_rratio 0.25)
+      (net 14 "LED_DIN"))
   )
   (footprint "carrier:XIAO-RP2040_preSoldered_header" (version 20240108) (generator generate_pcb.py) (layer "B.Cu")
@@
       (net 13 "LED_DATA"))
     (pad "2" thru_hole circle (at 5.0 0) (size 1.6 1.6) (drill 0.8) (layers *.Cu *.Mask)
-      (net 14 "LED_A"))
-  )
-  (footprint "carrier:THT_passive" (version 20240108) (generator generate_pcb.py) (layer "F.Cu")
+      (net 14 "LED_DIN"))
+  )
+  (footprint "carrier:THT_passive" (version 20240108) (generator generate_pcb.py) (layer "F.Cu")
